File: ECAD_main/ECAD_main.kicad_sch (KiCad schematic)
At the start: 0 parts

Commit message: Добавлена схема, сделана трассировка
Parts:
- added BL1: Photodiode, BPW34, symbol GOST_lib:root_1_Photodiode_GOST_lib.SchLib
- added C1, C3, C4: Capacitor, C1206, symbol GOST_lib:root_1_Capacitor_GOST_lib.SchLib
- added C2: Capacitor, C1206, symbol GOST_lib:root_2_Capacitor_GOST_lib.SchLib
- added DD1: TLV6001IDBVT, TLV6001, symbol GOST_lib:root_0_TLV6001IDBVT_GOST_lib.SchLib
- added HL1, HL2: LED, VSMY2850RG, symbol GOST_lib:root_3_LED_GOST_lib.SchLib
- added R1, R4: Resistor, R0603, symbol GOST_lib:root_0_Resistor_GOST_lib.SchLib
- added R10, R9: Resistor, R0603, symbol GOST_lib:root_2_Resistor_GOST_lib.SchLib
- added R2, R3, R5, R7, R8: Resistor, R0603, symbol GOST_lib:root_1_Resistor_GOST_lib.SchLib
- added R6: Resistor, R0603, symbol GOST_lib:root_3_Resistor_GOST_lib.SchLib
- added VT1, VT2: IRLML6244TRPBF, IRLML, symbol GOST_lib:root_0_IRLML6244TRPBF_GOST_lib.SchLib
Connections:
- new net: HL1.1, R3.1
- new net: HL1.2, VT1.3 (D)
- new net: C2.1, C4.2, DD1.1, R10.2, R9.1
- new net: BL1.2, C2.2, DD1.4, R9.2
- new net: R1.2, R2.2, VT1.1 (G)
- new net: HL2.1, R6.2
- new net: DD1.3, R7.2, R8.1
- new net: R4.2, R5.2, VT2.1 (G)
- new net: HL2.2, VT2.3 (D)
- new net +5: C1.2, C3.2, DD1.5 (+U), R3.2, R6.1, R8.2
- new net GND: BL1.1, C1.1, C3.1, C4.1, DD1.2 (-U), R2.1, R5.1, R7.1, VT1.2 (S), VT2.2 (S)
- new net IN: R1.1, R4.1
- new net OUT: R10.1
Other:
- company: МГТУ им. Н.Э.Баумана -> (none)
